Commit message: adding camera stuff and necessary gazebo information

File: my_robot_description/urdf/camera.xacro (robot description, xacro)
@@ -14,5 +14,5 @@
     </link>
     <joint name="camera_joint" type="fixed">
-        <!-- <axis xyz="0 1 0"/> -->
+        <axis xyz="0 1 0"/>
         <origin xyz="0.4 0 0.075" rpy="0 0 0"/>
         <parent link="chassis"/>
@@ -22,3 +22,43 @@
     	<material>Gazebo/DarkYellow</material>
     </gazebo>
+     <!-- camera -->
+    <gazebo reference="camera_link">
+        <sensor type="camera" name="camera_sensor">
+          <update_rate>30.0</update_rate>
+          <camera name="head">
+            <horizontal_fov>1.3962634</horizontal_fov>
+            <image>
+              <width>800</width>
+              <height>800</height>
+              <format>R8G8B8</format>
+            </image>
+            <clip>
+              <near>0.02</near>
+              <far>300</far>
+            </clip>
+            <noise>
+              <type>gaussian</type>
+              <!-- Noise is sampled independently per pixel on each frame.
+                   That pixel's noise value is added to each of its color
+                   channels, which at that point lie in the range [0,1]. -->
+              <mean>0.0</mean>
+              <stddev>0.007</stddev>
+            </noise>
+          </camera>
+          <plugin name="camera_controller" filename="libgazebo_ros_camera.so">
+            <alwaysOn>true</alwaysOn>
+            <updateRate>0.0</updateRate>
+            <cameraName>my_robot_camera</cameraName>
+            <imageTopicName>image_raw</imageTopicName>
+            <cameraInfoTopicName>camera_info</cameraInfoTopicName>
+            <frameName>camera_link</frameName>
+            <hackBaseline>0.07</hackBaseline>
+            <distortionK1>0.0</distortionK1>
+            <distortionK2>0.0</distortionK2>
+            <distortionK3>0.0</distortionK3>
+            <distortionT1>0.0</distortionT1>
+            <distortionT2>0.0</distortionT2>
+          </plugin>
+        </sensor>
+    </gazebo>
 </robot>
