Commit message: updated the launch files for gazebo and added imu stuff

File: my_robot_description/urdf/base.xacro (robot description, xacro)
@@ -44,3 +44,40 @@
         <material>Gazebo/Red</material>
     </gazebo>
+    <link name="imu_link" />
+    <joint name="imu_joint" type="fixed">
+        <origin xyz="0.4 0.0 0.001" rpy="0.0 0.0 0.0"/>
+        <parent link="base_link"/>
+        <child link="imu_link"/>
+        <axis xyz="0.0 0.0 0.0"/>
+    </joint>
+    <gazebo>
+        <plugin name="imu_plugin" filename="libgazebo_ros_imu.so">
+          <alwaysOn>true</alwaysOn>
+          <bodyName>chassis</bodyName>
+          <topicName>imu</topicName>
+          <serviceName>imu_service</serviceName>
+          <gaussianNoise>0.0</gaussianNoise>
+          <updateRate>20.0</updateRate>
+        </plugin>
+    </gazebo>
+    <gazebo reference="imu_link">
+        <gravity>true</gravity>
+        <sensor name="imu_sensor" type="imu">
+          <always_on>true</always_on>
+          <update_rate>100</update_rate>
+          <visualize>true</visualize>
+          <topic>__default_topic__</topic>
+          <plugin filename="libgazebo_ros_imu_sensor.so" name="imu_plugin">
+            <topicName>imu</topicName>
+            <bodyName>imu_link</bodyName>
+            <updateRateHZ>10.0</updateRateHZ>
+            <gaussianNoise>0.0</gaussianNoise>
+            <xyzOffset>0 0 0</xyzOffset>
+            <rpyOffset>0 0 0</rpyOffset>
+            <frameName>imu_link</frameName>
+            <initialOrientationAsReference>false</initialOrientationAsReference>
+          </plugin>
+          <pose>0 0 0 0 0 0</pose>
+        </sensor>
+    </gazebo>
 </robot>

Commit message: adding gmapping, navigation, and downsizing robot

File: my_robot_description/urdf/base.xacro (robot description, xacro)
@@ -15,9 +15,9 @@
     </xacro:macro>
     <link name="chassis">
-        <xacro:inertial_box mass="${body_mass}" x="0.8" y="0.7" z="0.1" />
+        <xacro:inertial_box mass="${body_mass}" x="0.5" y="0.3" z="0.1" />
         <visual>
             <origin xyz="0.0 0.0 0.075" rpy="0.0 0.0 0.0"/>
             <geometry>
-                <box size="0.8 0.7 0.15"/>
+                <box size="0.5 0.3 0.10"/>
             </geometry>
             <material name="">
@@ -29,10 +29,10 @@
             <origin xyz="0.0 0.0 0.075" rpy="0.0 0.0 0.0"/>
             <geometry>
-                <box size="0.8 0.7 0.15"/>
+                <box size="0.5 0.3 0.10"/>
             </geometry>
         </collision>
     </link>
     <joint name="base_joint" type="fixed">
-        <origin xyz="0.4 0.0 0.0" rpy="0.0 0.0 0.0"/>
+        <origin xyz="0.25 0.0 0.0" rpy="0.0 0.0 0.0"/>
         <parent link="base_link"/>
         <child link="chassis"/>
@@ -40,11 +40,11 @@
     </joint>
     <gazebo reference="chassis">
-        <mu1>0.2</mu1>
-        <mu2>0.2</mu2>
+        <mu1>0.1</mu1>
+        <mu2>0.1</mu2>
         <material>Gazebo/Red</material>
     </gazebo>
     <link name="imu_link" />
     <joint name="imu_joint" type="fixed">
-        <origin xyz="0.4 0.0 0.001" rpy="0.0 0.0 0.0"/>
+        <origin xyz="0.25 0.0 0.03" rpy="0.0 0.0 0.0"/>
         <parent link="base_link"/>
         <child link="imu_link"/>
@@ -56,4 +56,5 @@
           <bodyName>chassis</bodyName>
           <topicName>imu</topicName>
+          <frameName>chassis</frameName>
           <serviceName>imu_service</serviceName>
           <gaussianNoise>0.0</gaussianNoise>

File: my_robot_description/urdf/camera.xacro (robot description, xacro)
@@ -5,5 +5,5 @@
             <origin xyz="0 0 0" rpy="0 0 0"/>
             <geometry>
-                <box size="0.03 0.1 0.1"/>
+                <box size="0.03 0.08 0.05"/>
             </geometry>
             <material name="yellow">
@@ -15,5 +15,5 @@
     <joint name="camera_joint" type="fixed">
         <axis xyz="0 1 0"/>
-        <origin xyz="0.4 0 0.075" rpy="0 0 0"/>
+        <origin xyz="0.25 0 0.075" rpy="0 0 0"/>
         <parent link="chassis"/>
         <child link="camera_link"/>

File: my_robot_description/urdf/my_wheel.xacro (robot description, xacro)
@@ -29,5 +29,5 @@
                 <origin xyz="0.0 0.0 0.0" rpy="0.0 0.0 0.0"/>
                 <geometry>
-                    <mesh filename="${file_path}" scale="0.005 0.005 0.005"/>
+                    <mesh filename="${file_path}" scale="0.003 0.003 0.003"/>
                 </geometry>
                 <material name="black">
@@ -47,18 +47,18 @@
             <child link="wheel_${name}_link"/>
             <axis xyz="0 1 0"/>
-            <limit effort="100.0" lower="-10.0" upper="10.0" velocity="10"/>
-            <dynamics damping="0.1" friction="0.9"/>
+            <limit effort="50.0" lower="-10.0" upper="10.0" velocity="10"/>
+            <dynamics damping="0.3" friction="1.0"/>
         </joint>
         <gazebo reference="wheel_${name}_link">
-            <mu1>0.2</mu1>
-            <mu2>0.2</mu2>
+            <mu1>0.1</mu1>
+            <mu2>0.1</mu2>
             <material>Gazebo/Black</material>
         </gazebo>
     </xacro:macro>
     <!-- Creating wheels using macros template -->
-    <xacro:wheel name="rear_right"  x="0.250" y ="0.40" file_path="package://my_robot_description/meshes/right_tire.stl" />
-    <xacro:wheel name="front_right" x="-0.250" y ="0.40" file_path="package://my_robot_description/meshes/right_tire.stl" />
-    <xacro:wheel name="front_left"  x="-0.250" y ="-0.40" file_path="package://my_robot_description/meshes/left_tire.stl" />
-    <xacro:wheel name="rear_left"   x="0.250" y ="-0.40" file_path="package://my_robot_description/meshes/left_tire.stl" />
+    <xacro:wheel name="rear_right"  x="0.150" y ="0.18" file_path="package://my_robot_description/meshes/right_tire.stl" />
+    <xacro:wheel name="front_right" x="-0.150" y ="0.18" file_path="package://my_robot_description/meshes/right_tire.stl" />
+    <xacro:wheel name="front_left"  x="-0.150" y ="-0.18" file_path="package://my_robot_description/meshes/left_tire.stl" />
+    <xacro:wheel name="rear_left"   x="0.150" y ="-0.18" file_path="package://my_robot_description/meshes/left_tire.stl" />
     <!-- wheel_${name}_joint -->
     <!-- adding skid controller essential for teleop and navigation -->

Commit message: updating files to deal with gazebo dynamics

File: my_robot_description/urdf/base.xacro (robot description, xacro)
@@ -40,6 +40,6 @@
     </joint>
     <gazebo reference="chassis">
-        <mu1>0.1</mu1>
-        <mu2>0.1</mu2>
+        <mu1>0.002</mu1>
+        <mu2>0.002</mu2>
         <material>Gazebo/Red</material>
     </gazebo>

File: my_robot_description/urdf/lidar_sensor.xacro (robot description, xacro)
@@ -57,6 +57,6 @@
     </joint>
     <gazebo reference="sensor_mount">
-        <mu1>0.2</mu1>
-        <mu2>0.2</mu2>
+        <!-- <mu1>0.2</mu1>
+        <mu2>0.2</mu2> -->
         <material>Gazebo/Blue</material>
     </gazebo>

File: my_robot_description/urdf/my_wheel.xacro (robot description, xacro)
@@ -6,11 +6,11 @@
     <!-- assuming wheels to be of a hypothetical material with density 15 -->
     <xacro:property name="wheel_density" value="15"/>
-    <xacro:property name="wheel_radius" value="0.15"/>
-    <xacro:property name="wheel_length" value="0.1"/>
+    <xacro:property name="wheel_radius" value="0.1"/>
+    <xacro:property name="wheel_length" value="0.08"/>
     <xacro:property name="pi" value="3.141592654"/>
     <xacro:property name="body_mass" value="10"/>
     <xacro:property name="wheel_mass" value="${wheel_density*pi*wheel_radius*wheel_radius*wheel_length}"/>
     <xacro:property name="Iz_wheel" value="${0.5*wheel_mass*wheel_radius*wheel_radius}" />
-    <xacro:property name="I_wheel" value="${(1.0/12.0)*wheel_mass*(3.0*wheel_radius*wheel_radius+wheel_length*wheel_length)}"/>
+    <xacro:property name="I_wheel" value="${(1.0/12.0)*wheel_mass*(3.0*wheel_radius*wheel_radius + wheel_length*wheel_length)}"/>
     <!-- creating the inertial macros -->
     <xacro:macro name="inertia_wheel">
@@ -47,10 +47,12 @@
             <child link="wheel_${name}_link"/>
             <axis xyz="0 1 0"/>
-            <limit effort="50.0" lower="-10.0" upper="10.0" velocity="10"/>
-            <dynamics damping="0.3" friction="1.0"/>
+            <!-- <limit effort="10.0" velocity="1"/> -->
+            <!-- <dynamics damping="0.2" friction="0.1"/> -->
         </joint>
         <gazebo reference="wheel_${name}_link">
-            <mu1>0.1</mu1>
-            <mu2>0.1</mu2>
+            <mu1>0.4</mu1>
+            <mu2>0.4</mu2>
+            <kp>1000.0</kp>
+            <kd>0.75</kd>
             <material>Gazebo/Black</material>
         </gazebo>
@@ -65,5 +67,5 @@
     <gazebo>
         <plugin name="skid_steer_drive_controller" filename="libgazebo_ros_skid_steer_drive.so">
-            <updateRate>100.0</updateRate>
+            <updateRate>1000.0</updateRate>
             <robotNamespace>/</robotNamespace>
             <!-- <ros><remap from="odom" to="/odom"/></ros> -->
@@ -72,8 +74,8 @@
             <leftRearJoint>wheel_rear_left_joint</leftRearJoint>
             <rightRearJoint>wheel_rear_right_joint</rightRearJoint>
-            <wheelSeparation>0.8</wheelSeparation>
+            <wheelSeparation>0.6</wheelSeparation>
             <wheelDiameter>${2 * wheel_radius}</wheelDiameter>
             <robotBaseFrame>base_footprint</robotBaseFrame>
-            <torque>50</torque>
+            <torque>1000</torque>
             <!-- for sending command messages (twist) -->
             <!-- <topicName>cmd_vel</topicName> -->
