Commit message: updating entire positioning of origin for robot components

File: line_robt_follower/urdf/line_robt_follower.urdf (robot description, URDF)
Before this commit: robot line_robt_follower, 6 links, 5 joints
Links:
- removed link base_link
- added link chassis, mass 0.10052; collision mesh filename=package://line_robt_follower/meshes/chassis.STL scale=1 1 1; visual mesh filename=package://line_robt_follower/meshes/chassis.STL scale=1 1 1
Joints:
- joint base_joint: child base_link -> chassis
- joint castorjoint: parent base_link -> chassis
- joint leftwheel: parent base_link -> chassis
- joint rightwheel: parent base_link -> chassis

File: my_robot_description/urdf/base.xacro (robot description, xacro)
@@ -1,5 +1,5 @@
 <?xml version="1.0"?>
 <robot xmlns:xacro="http://www.ros.org/wiki/xacro">
-    <link name="base_footprint" />
+    <link name="base_link" />
     <!-- body attributes -->
     <xacro:property name="body_mass" value="2.0"/>
@@ -14,10 +14,10 @@
         </inertial>
     </xacro:macro>
-    <link name="base_link">
+    <link name="chassis">
         <xacro:inertial_box mass="${body_mass}" x="0.8" y="0.7" z="0.1" />
-        <visual name="">
-            <origin xyz="0.0 0.0 0.0" rpy="0.0 0.0 0.0"/>
+        <visual>
+            <origin xyz="0.0 0.0 0.075" rpy="0.0 0.0 0.0"/>
             <geometry>
-                <box size="0.8 0.7 0.2"/>
+                <box size="0.8 0.7 0.15"/>
             </geometry>
             <material name="">
@@ -27,17 +27,17 @@
         </visual>
         <collision>
-            <origin xyz="0.0 0.0 0.0" rpy="0.0 0.0 0.0"/>
+            <origin xyz="0.0 0.0 0.075" rpy="0.0 0.0 0.0"/>
             <geometry>
-                <box size="0.0 0.0 0.0"/>
+                <box size="0.8 0.7 0.15"/>
             </geometry>
         </collision>
     </link>
     <joint name="base_joint" type="fixed">
-        <origin xyz="0.0 0.0 0.135" rpy="0.0 0.0 0.0"/>
-        <parent link="base_footprint"/>
-        <child link="base_link"/>
+        <origin xyz="0.4 0.0 0.0" rpy="0.0 0.0 0.0"/>
+        <parent link="base_link"/>
+        <child link="chassis"/>
         <axis xyz="0.0 0.0 0.0"/>
     </joint>
-    <gazebo reference="base_link">
+    <gazebo reference="chassis">
         <mu1>0.2</mu1>
         <mu2>0.2</mu2>

File: my_robot_description/urdf/camera.xacro (robot description, xacro)
@@ -7,10 +7,14 @@
                 <box size="0.03 0.1 0.1"/>
             </geometry>
+            <material name="yellow">
+            	<color rgba="1.0 0.92 0.016 1.0"/>
+                <texture filename=""/>
+            </material>
         </visual>
     </link>
     <joint name="camera_joint" type="fixed">
         <!-- <axis xyz="0 1 0"/> -->
-        <origin xyz="0.4 0 0" rpy="0 0 0"/>
-        <parent link="base_link"/>
+        <origin xyz="0.4 0 0.075" rpy="0 0 0"/>
+        <parent link="chassis"/>
         <child link="camera_link"/>
     </joint>

File: my_robot_description/urdf/lidar_sensor.xacro (robot description, xacro)
@@ -4,9 +4,9 @@
         <inertial>
             <mass value="1e-5" />
-            <origin xyz="0 0 0" rpy="0 0 0"/>
+            <origin xyz="0 0 0.16" rpy="0 0 0"/>
             <inertia ixx="1e-6" ixy="0" ixz="0" iyy="1e-6" iyz="0" izz="1e-6" />
         </inertial>
         <visual>
-            <origin xyz="0 0 0" rpy="0 0 0"/>
+            <origin xyz="0 0 0.0" rpy="0 0 0"/>
             <material name="">
                 <color rgba="0.0 0.0 1.0 1.0"/>
@@ -14,5 +14,5 @@
             </material>
             <geometry>
-                <box size="0.1 0.1 0.1"/>
+                <box size="0.1 0.1 0.05"/>
             </geometry>
         </visual>
@@ -25,6 +25,6 @@
     </link>
     <joint name="sensor_mount_joint" type="fixed">
-        <origin xyz="0.0 0.0 0.1" rpy="0.0 0.0 0.0"/>
-        <parent link="base_link"/>
+        <origin xyz="0.0 0.0 0.15" rpy="0.0 0.0 0.0"/>
+        <parent link="chassis"/>
         <child link="sensor_mount"/>
         <axis xyz="0.0 0.0 0.0"/>
@@ -44,5 +44,5 @@
         </visual>
         <collision>
-            <origin xyz="0.0 0.0 0.0" rpy="0.0 0.0 0.0"/>
+            <origin xyz="0.0 0.0 0" rpy="0.0 0.0 0.0"/>
             <geometry>
                 <box size="0.1 0.1 0.1"/>
@@ -52,5 +52,5 @@
     <joint name="hokuyo_joint" type="fixed">
         <axis xyz="0 1 0"/>
-        <origin xyz="0 0 0.08" rpy="0 0 0"/>
+        <origin xyz="0 0 0.05" rpy="0 0 0"/>
         <parent link="sensor_mount"/>
         <child link="hokuyo_lidar"/>

File: my_robot_description/urdf/my_robot_assembly.xacro (robot description, xacro)
@@ -5,6 +5,4 @@
     <!-- importing the template for the robot wheels -->
     <xacro:include filename="$(find my_robot_description)/urdf/my_wheel.xacro"/>
-    <!-- importing all the related gazebo configurations -->
-    <!-- <xacro:include filename="$(find my_robot_description)/urdf/gazebo.xacro"/> -->
     <!-- Macros for importing the lidar -->
     <xacro:include filename="$(find my_robot_description)/urdf/lidar_sensor.xacro"/>

File: my_robot_description/urdf/my_wheel.xacro (robot description, xacro)
@@ -43,10 +43,10 @@
         </link>
         <joint name="wheel_${name}_joint" type="continuous">
-            <origin xyz="${x} ${y} .0" rpy="0 0.0 0.0"/>
-            <parent link="base_link"/>
+            <origin xyz="${x} ${y} 0.075" rpy="0 0.0 0.0"/>
+            <parent link="chassis"/>
             <child link="wheel_${name}_link"/>
             <axis xyz="0 1 0"/>
-            <limit effort="100.0" velocity="100.0"/>
-            <dynamics damping="1.0" friction="1.0"/>
+            <limit effort="100.0" lower="-10.0" upper="10.0" velocity="10"/>
+            <dynamics damping="0.1" friction="0.9"/>
         </joint>
         <gazebo reference="wheel_${name}_link">
